File: M0116/M0116.kicad_sch (KiCad schematic)
At the start: 2 parts, among them J2 Conn_01x04

Commit message: switched D+/D- on USB PCB, isolated shield from ground
Connections:
- net GND: no longer ADB-FEM1.5 (SH), ADB-FEM1.6 (SH), ADB-FEM1.7 (SH)
- new net: ADB-FEM1.5 (SH), ADB-FEM1.6 (SH), ADB-FEM1.7 (SH)
- no-connect marks 0 -> 1
Changed lines of the file:
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@@
 (kicad_sch (version 20230121) (generator eeschema)
   (paper "A4")
+  (no_connect (at 54.61 33.02))
   (wire (pts (xy 29.21 33.02) (xy 31.75 33.02))
     (stroke (width 0) (type default))
@@
     (pin "4")
     (instances
-      (project "aekii-m3501"
+      (project "M0116"
         (path "/10fa40d7-dfa7-4104-a535-2d62cfab9a1c"
           (reference "J2") (unit 1)
@@
     (pin "1")
     (instances
-      (project "aekii-m3501"
+      (project "M0116"
         (path "/10fa40d7-dfa7-4104-a535-2d62cfab9a1c"
           (reference "#PWR03") (unit 1)
@@
     (pin "7")
     (instances
-      (project "aekii-m3501"
+      (project "M0116"
         (path "/10fa40d7-dfa7-4104-a535-2d62cfab9a1c"
           (reference "ADB-FEM1") (unit 1)
@@
     (pin "1")
     (instances
-      (project "aekii-m3501"
+      (project "M0116"
         (path "/10fa40d7-dfa7-4104-a535-2d62cfab9a1c"
           (reference "#PWR01") (unit 1)
         )
       )
-    )
-  )
-  (symbol (lib_id "power:GND") (at 54.61 33.02 0) (unit 1)
-    (in_bom yes) (on_board yes) (dnp no) (fields_autoplaced)
-    (property "Reference" "#PWR02" (at 54.61 39.37 0)
-      (effects (font (size 1.27 1.27)) hide)
-    )
-    (property "Value" "GND" (at 54.61 38.1 0)
-      (effects (font (size 1.27 1.27)))
-    )
-    (property "Footprint" "" (at 54.61 33.02 0)
-      (effects (font (size 1.27 1.27)) hide)
-    )
-    (property "Datasheet" "" (at 54.61 33.02 0)
-      (effects (font (size 1.27 1.27)) hide)
-    )
-    (pin "1")
-    (instances
-      (project "aekii-m3501"
-        (path "/10fa40d7-dfa7-4104-a535-2d62cfab9a1c"
-          (reference "#PWR02") (unit 1)
-        )
-      )
